Commit message: RPP

File: src/mecanum_robot_sim/urdf/mecanum_robot.urdf.xacro (robot description, xacro)
@@ -231,36 +231,15 @@
   </gazebo>
   <!-- ═══════════════════════════════════════════════════════════════
-       ros2_control  —  velocity interface for 4 wheels
-  ═══════════════════════════════════════════════════════════════ -->
-  <ros2_control name="GazeboSimSystem" type="system">
-    <hardware>
-      <plugin>gz_ros2_control/GazeboSimSystem</plugin>
-    </hardware>
-    <joint name="front_left_wheel_joint">
-      <command_interface name="velocity"><param name="min">-10</param><param name="max">10</param></command_interface>
-      <state_interface name="position"/><state_interface name="velocity"/>
-    </joint>
-    <joint name="front_right_wheel_joint">
-      <command_interface name="velocity"><param name="min">-10</param><param name="max">10</param></command_interface>
-      <state_interface name="position"/><state_interface name="velocity"/>
-    </joint>
-    <joint name="rear_left_wheel_joint">
-      <command_interface name="velocity"><param name="min">-10</param><param name="max">10</param></command_interface>
-      <state_interface name="position"/><state_interface name="velocity"/>
-    </joint>
-    <joint name="rear_right_wheel_joint">
-      <command_interface name="velocity"><param name="min">-10</param><param name="max">10</param></command_interface>
-      <state_interface name="position"/><state_interface name="velocity"/>
-    </joint>
-  </ros2_control>
-  <!-- gz_ros2_control system plugin -->
+       Kinematic body-velocity control
+       VelocityControl directly sets the model's body-frame velocity,
+       bypassing wheel contact physics (which cannot simulate mecanum
+       lateral motion with sphere collision proxies).
+       cmd_vel_relay converts /cmd_vel (TwistStamped) → /cmd_vel_gz
+       (Twist), which is bridged here from ROS → Ignition.
+  ═══════════════════════════════════════════════════════════════ -->
   <gazebo>
-    <plugin filename="gz_ros2_control-system"
-            name="gz_ros2_control::GazeboSimROS2ControlPlugin">
-      <parameters>$(find mecanum_robot_sim)/config/mecanum_drive_controller.yaml</parameters>
-      <ros>
-        <remapping>/mecanum_drive_controller/reference:=/cmd_vel</remapping>
-        <remapping>/mecanum_drive_controller/odom:=/odom</remapping>
-      </ros>
+    <plugin filename="ignition-gazebo-velocity-control-system"
+            name="ignition::gazebo::systems::VelocityControl">
+      <topic>/cmd_vel_gz</topic>
     </plugin>
   </gazebo>

Commit message: update local cost map, global
🔥 update global cost map (dummy straight line), local costmap w/o human detection

File: src/mecanum_robot_sim/urdf/mecanum_robot.urdf.xacro (robot description, xacro)
@@ -110,5 +110,5 @@
   </link>
   <joint name="lidar_joint" type="fixed">
-    <origin xyz="0 0 0.22" rpy="0 0 0"/>
+    <origin xyz="0 0 0.40" rpy="0 0 0"/>
     <parent link="base_link"/>
     <child link="lidar_link"/>

Commit message: update local cost map, global
🔥 update global cost map (dummy straight line), local costmap w/o human detection

File: src/mecanum_robot_sim/urdf/mecanum_robot.urdf.xacro (robot description, xacro)
@@ -110,5 +110,5 @@
   </link>
   <joint name="lidar_joint" type="fixed">
-    <origin xyz="0 0 0.4" rpy="0 0 0"/>
+    <origin xyz="0 0 0.22" rpy="0 0 0"/>
     <parent link="base_link"/>
     <child link="lidar_link"/>

Commit message: Refactor: Human Detection

File: src/mecanum_robot_sim/urdf/mecanum_robot.urdf.xacro (robot description, xacro)
@@ -110,5 +110,5 @@
   </link>
   <joint name="lidar_joint" type="fixed">
-    <origin xyz="0 0 0.22" rpy="0 0 0"/>
+    <origin xyz="0 0 0.4" rpy="0 0 0"/>
     <parent link="base_link"/>
     <child link="lidar_link"/>

Commit message: Refactor: something

File: src/mecanum_robot_sim/urdf/mecanum_robot.urdf.xacro (robot description, xacro)
@@ -158,5 +158,5 @@
   <!-- mounted at front face (x=+0.40), 0.18 m above base_link origin -->
   <joint name="camera_joint" type="fixed">
-    <origin xyz="0.40 0 0.18" rpy="0 0 0"/>
+    <origin xyz="0.40 0 0.5" rpy="0 0 0"/>
     <parent link="base_link"/>
     <child link="camera_link"/>

Commit message: Update

File: src/mecanum_robot_sim/urdf/mecanum_robot.urdf.xacro (robot description, xacro)
@@ -110,5 +110,5 @@
   </link>
   <joint name="lidar_joint" type="fixed">
-    <origin xyz="0 0 0.22" rpy="0 0 0"/>
+    <origin xyz="0 0 0.4" rpy="0 0 0"/>
     <parent link="base_link"/>
     <child link="lidar_link"/>
@@ -158,5 +158,5 @@
   <!-- mounted at front face (x=+0.40), 0.18 m above base_link origin -->
   <joint name="camera_joint" type="fixed">
-    <origin xyz="0.40 0 0.18" rpy="0 0 0"/>
+    <origin xyz="0.40 0 0.5" rpy="0 0 0"/>
     <parent link="base_link"/>
     <child link="camera_link"/>
